Commit message: Adds duckiebot visualization in rviz

File: catkin_ws/src/duckietown_description/urdf/duckiebot.urdf.xacro (robot description, xacro)
@@ -3,6 +3,7 @@
     <link name="duckiebot">
         <visual>
+            <origin xyz="0 0 0.04" />
             <geometry>
-                <box size="0.3 0.3 0.3" />
+                <mesh filename="package://duckietown_description/urdf/meshes/duckiebot.dae" />
             </geometry>
         </visual>
