Commit message: replaces stop sign to tag_id in macros file

File: catkin_ws/src/duckietown_description/urdf/macros.urdf.xacro (robot description, xacro)
@@ -27,5 +27,5 @@
                 <origin xyz="-0.0254 -0.0254 0" />
                 <geometry>
-                    <mesh filename="package://duckietown_description/urdf/meshes/sign_stop.dae" />
+                    <mesh filename="package://duckietown_description/urdf/meshes/tags/tag_${id}.dae" />
                 </geometry>
             </visual>

Commit message: fixes the tag_${id}.dae reference

File: catkin_ws/src/duckietown_description/urdf/macros.urdf.xacro (robot description, xacro)
@@ -27,5 +27,5 @@
                 <origin xyz="-0.0254 -0.0254 0" />
                 <geometry>
-                    <mesh filename="package://duckietown_description/urdf/meshes/tags/tag_${id}.dae" />
+                    <mesh filename="package://duckietown_description/urdf/meshes/tag_${id}.dae" />
                 </geometry>
             </visual>
